File: esdm/esdm.kicad_pcb (KiCad board)
At the start: 2 copper layers, 54 x 23.3 mm, 11 parts, among them J1 Barrel_Jack, J2 Conn_02x02_Odd_Even, J3 Conn_02x02_Odd_Even, U1 AZ1117-3.3, U2 AZ1117-5.0

Commit message: rearranged directory
Routing:
- added copper zone on B.Cu, net GND
- added copper zone on F.Cu, net GND
Changed lines of the file:
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@@
-(kicad_pcb (version 20171130) (host pcbnew "(5.1.5)-3")
+(kicad_pcb (version 20171130) (host pcbnew 5.1.5-52549c5~84~ubuntu18.04.1)
   (general
     (thickness 1.6)
@@
       (outputformat 1)
       (mirror false)
-      (drillshape 1)
+      (drillshape 0)
       (scaleselection 1)
-      (outputdirectory ""))
+      (outputdirectory "./"))
   )
   (net 0 "")
@@
   (segment (start 145.06 72.6) (end 146.41 71.25) (width 0.25) (layer F.Cu) (net 5))
   (segment (start 144.485 72.6) (end 145.06 72.6) (width 0.25) (layer F.Cu) (net 5))
+  (zone (net 2) (net_name GND) (layer F.Cu) (hatch edge 0.508)
+    (connect_pads (clearance 0.508))
+    (min_thickness 0.254)
+    (fill yes (arc_segments 32) (thermal_gap 0.508) (thermal_bridge_width 0.508))
+    (polygon
+      (pts
+        (xy 175.26 81.28) (xy 106.68 81.28) (xy 106.68 50.8) (xy 175.26 50.8)
+      )
+    )
+  )
+  (zone (net 2) (net_name GND) (layer B.Cu) (hatch edge 0.508)
+    (connect_pads (clearance 0.508))
+    (min_thickness 0.254)
+    (fill yes (arc_segments 32) (thermal_gap 0.508) (thermal_bridge_width 0.508))
+    (polygon
+      (pts
+        (xy 176.53 82.55) (xy 105.41 82.55) (xy 105.41 49.53) (xy 176.53 49.53)
+      )
+    )
+  )
 )
