File: vga_controller/vga_controller/decoder_circuit.sch (KiCad schematic (older format))
At the start: 0 parts

Commit message: d
Parts:
- added U1, U2: CAT28C16AL-20, CAT28C16AL-20:DIP254P1524X635-24, symbol CAT28C16AL-20:CAT28C16AL-20
- added U3, U4: 7400, CD4011BE:DIP254P762X508-14, symbol 74xx:7400
Connections:
- new net: U1.10 (I/O1), U3.9
- new net: U1.11 (I/O2), U3.13
- new net: U1.13 (I/O3), U3.4
- new net: U1.9 (I/O0), U3.2
- new net: U2.14 (I/O4), U4.4
- new net: U2.15 (I/O5), U4.9
- new net: U2.16 (I/O6), U4.13
- new net: U2.17 (I/O7), U4.2
- new net: U3.1, U3.6
- new net: U3.10, U3.11
- new net: U4.1, U4.6
- new net: U4.10, U4.11
- new net +5V: U1.21 (~WE), U1.24 (VCC), U2.21 (~WE), U2.24 (VCC), U3.14 (VCC), U4.14 (VCC)
- new net GND: U1.12 (VSS), U1.18 (~CE), U1.20 (~OE), U2.12 (VSS), U2.18 (~CE), U2.20 (~OE), U3.7 (GND), U4.7 (GND)
- new net H_BLANK: U3.3, U3.5
- new net H_SYNC: U3.12, U3.8
- new net V_BLANK: U4.3, U4.5
- new net V_SYNC: U4.12, U4.8
- new net x0: U1.8 (A0)
- new net x1: U1.7 (A1)
- new net x2: U1.6 (A2)
- new net x3: U1.5 (A3)
- new net x4: U1.4 (A4)
- new net x5: U1.3 (A5)
- new net x6: U1.2 (A6)
- new net x7: U1.1 (A7)
- new net x8: U1.23 (A8)
- new net y0: U2.8 (A0)
- new net y1: U2.7 (A1)
- new net y2: U2.6 (A2)
- new net y3: U2.5 (A3)
- new net y4: U2.4 (A4)
- new net y5: U2.3 (A5)
- new net y6: U2.2 (A6)
- new net y7: U2.1 (A7)
- new net y8: U2.23 (A8)
- new net y9: U2.22 (A9)
- no-connect marks 0 -> 11
