File: vga_controller/vga_controller/decoder_circuit.sch (KiCad schematic (older format))
At the start: 4 parts, among them U1 CAT28C16AL-20, U2 CAT28C16AL-20, U3 7400, U4 7400

Commit message: made interconnections between sheets
Connections:
- net x-reset: now reaches U1.13 (I/O3), U3.4
- net y-reset: now reaches U2.17 (I/O7), U4.2
Changed lines of the file:
@@
 EESchema Schematic File Version 4
-LIBS:vga_controller-cache
-EELAYER 26 0
+EELAYER 30 0
 EELAYER END
 $Descr A4 11693 8268
@@
 	3950 1200 5500 1200
 Wire Wire Line
-	6700 2400 7000 2400
-Wire Wire Line
 	3950 1300 5250 1300
 Wire Wire Line
@@
 NoConn ~ 3950 1800
 NoConn ~ 3950 1900
-Wire Wire Line
-	6700 1750 7000 1750
-Text HLabel 7000 2400 2    50   Input ~ 0
-H_SYNC
-Text HLabel 7000 1750 2    50   Input ~ 0
-H_BLANK
-Connection ~ 6700 1750
-Connection ~ 6700 2400
 NoConn ~ 3950 4350
 NoConn ~ 3950 4450
@@
 	4150 3950 5850 3950
 Wire Wire Line
-	3950 5050 5300 5050
+	3950 5050 4150 5050
 Wire Wire Line
 	5300 5050 5300 4950
@@
 	6750 5500 7000 5500
 Connection ~ 6750 5500
-Text HLabel 7000 4850 2    50   Input ~ 0
-V_BLANK
-Text HLabel 7000 5500 2    50   Input ~ 0
-V_SYNC
 $Comp
 L power:+5V #PWR05
@@
 NoConn ~ 2550 2800
 NoConn ~ 2550 5950
+Connection ~ 6700 2400
+Wire Wire Line
+	6700 2400 7000 2400
+Text HLabel 7000 2400 2    50   Output ~ 0
+H_SYNC
+Text HLabel 7000 4850 2    50   Output ~ 0
+V_BLANK
+Text HLabel 7000 5500 2    50   Output ~ 0
+V_SYNC
+Connection ~ 6700 1750
+Text HLabel 7000 1750 2    50   Output ~ 0
+H_BLANK
+Wire Wire Line
+	6700 1750 7000 1750
+Text GLabel 4150 1700 3    50   Output ~ 0
+x-reset
+Wire Wire Line
+	4150 1700 4150 1500
+Connection ~ 4150 1500
+Text GLabel 4150 5250 3    50   Output ~ 0
+y-reset
+Wire Wire Line
+	4150 5050 4150 5250
+Connection ~ 4150 5050
+Wire Wire Line
+	4150 5050 5300 5050
 $EndSCHEMATC

Commit message: added routes
Parts:
- U3, U4: footprint CD4011BE:DIP254P762X508-14 -> Package_DIP:DIP-14_W7.62mm
Changed lines of the file:
@@
 F 0 "U3" H 6100 1275 50  0000 C CNN
 F 1 "7400" H 6100 1184 50  0000 C CNN
-F 2 "CD4011BE:DIP254P762X508-14" H 6100 950 50  0001 C CNN
+F 2 "Package_DIP:DIP-14_W7.62mm" H 6100 950 50  0001 C CNN
 F 3 "http://www.ti.com/lit/gpn/sn7400" H 6100 950 50  0001 C CNN
 	2    6100 950
@@
 F 0 "U3" H 6100 2075 50  0000 C CNN
 F 1 "7400" H 6100 1984 50  0000 C CNN
-F 2 "CD4011BE:DIP254P762X508-14" H 6100 1750 50  0001 C CNN
+F 2 "Package_DIP:DIP-14_W7.62mm" H 6100 1750 50  0001 C CNN
 F 3 "http://www.ti.com/lit/gpn/sn7400" H 6100 1750 50  0001 C CNN
 	1    6100 1750
@@
 F 0 "U3" H 6100 2725 50  0000 C CNN
 F 1 "7400" H 6100 2634 50  0000 C CNN
-F 2 "CD4011BE:DIP254P762X508-14" H 6100 2400 50  0001 C CNN
+F 2 "Package_DIP:DIP-14_W7.62mm" H 6100 2400 50  0001 C CNN
 F 3 "http://www.ti.com/lit/gpn/sn7400" H 6100 2400 50  0001 C CNN
 	3    6100 2400
@@
 F 0 "U3" H 6100 3525 50  0000 C CNN
 F 1 "7400" H 6100 3434 50  0000 C CNN
-F 2 "CD4011BE:DIP254P762X508-14" H 6100 3200 50  0001 C CNN
+F 2 "Package_DIP:DIP-14_W7.62mm" H 6100 3200 50  0001 C CNN
 F 3 "http://www.ti.com/lit/gpn/sn7400" H 6100 3200 50  0001 C CNN
 	4    6100 3200
@@
 F 0 "U3" H 8230 1296 50  0000 L CNN
 F 1 "7400" H 8230 1205 50  0000 L CNN
-F 2 "CD4011BE:DIP254P762X508-14" H 8000 1250 50  0001 C CNN
+F 2 "Package_DIP:DIP-14_W7.62mm" H 8000 1250 50  0001 C CNN
 F 3 "http://www.ti.com/lit/gpn/sn7400" H 8000 1250 50  0001 C CNN
 	5    8000 1250
@@
 F 0 "U4" H 6150 4375 50  0000 C CNN
 F 1 "7400" H 6150 4284 50  0000 C CNN
-F 2 "CD4011BE:DIP254P762X508-14" H 6150 4050 50  0001 C CNN
+F 2 "Package_DIP:DIP-14_W7.62mm" H 6150 4050 50  0001 C CNN
 F 3 "http://www.ti.com/lit/gpn/sn7400" H 6150 4050 50  0001 C CNN
 	2    6150 4050
@@
 F 0 "U4" H 6150 5175 50  0000 C CNN
 F 1 "7400" H 6150 5084 50  0000 C CNN
-F 2 "CD4011BE:DIP254P762X508-14" H 6150 4850 50  0001 C CNN
+F 2 "Package_DIP:DIP-14_W7.62mm" H 6150 4850 50  0001 C CNN
 F 3 "http://www.ti.com/lit/gpn/sn7400" H 6150 4850 50  0001 C CNN
 	1    6150 4850
@@
 F 0 "U4" H 6150 5825 50  0000 C CNN
 F 1 "7400" H 6150 5734 50  0000 C CNN
-F 2 "CD4011BE:DIP254P762X508-14" H 6150 5500 50  0001 C CNN
+F 2 "Package_DIP:DIP-14_W7.62mm" H 6150 5500 50  0001 C CNN
 F 3 "http://www.ti.com/lit/gpn/sn7400" H 6150 5500 50  0001 C CNN
 	3    6150 5500
@@
 F 0 "U4" H 6150 6625 50  0000 C CNN
 F 1 "7400" H 6150 6534 50  0000 C CNN
-F 2 "CD4011BE:DIP254P762X508-14" H 6150 6300 50  0001 C CNN
+F 2 "Package_DIP:DIP-14_W7.62mm" H 6150 6300 50  0001 C CNN
 F 3 "http://www.ti.com/lit/gpn/sn7400" H 6150 6300 50  0001 C CNN
 	4    6150 6300
@@
 F 0 "U4" H 8280 4396 50  0000 L CNN
 F 1 "7400" H 8280 4305 50  0000 L CNN
-F 2 "CD4011BE:DIP254P762X508-14" H 8050 4350 50  0001 C CNN
+F 2 "Package_DIP:DIP-14_W7.62mm" H 8050 4350 50  0001 C CNN
 F 3 "http://www.ti.com/lit/gpn/sn7400" H 8050 4350 50  0001 C CNN
 	5    8050 4350
