File: vga_controller/vga_controller/vga_controller.sch (KiCad schematic (older format))
At the start: 8 parts, among them U11 CAT28C513-D, U12 7400

Commit message: made interconnections between sheets
Parts:
- removed R10, R12, R8: 1.5KΩ, symbol Device:R
- removed R11, R7, R9: 680Ω, symbol Device:R
- removed U11: CAT28C513-D, Package_DIP:DIP-32_W7.62mm, symbol parallel_eeprom:CAT28C513-D
- removed U12: 7400, symbol 74xx:7400
Connections:
- net labels removed: Blue, Green, H_BLANK, Red, V_BLANK, x0, x1, x2, x3, x4, x5, x6, x7, y0, y1, y2, y3, y4, y5, y6, y7
- wire segments 64 -> 117
- no-connect marks 2 -> 0
