File: vga_controller/vga_controller/counter_circuit.sch (KiCad schematic (older format))
At the start: 7 parts, among them U10 74LS161, U5 74LS161, U6 74LS161, U7 74LS161, U8 74LS161, U9 74LS161, X1 ACO-xxxMHz

Commit message: footprints
Parts:
- U10, U5, U6, U7, U8, U9: footprint (none) -> SN74LS161AD:SOIC127P600X175-16N
Changed lines of the file:
@@
 F 0 "U8" H 3750 4981 50  0000 C CNN
 F 1 "74LS161" H 3750 4890 50  0000 C CNN
-F 2 "" H 3750 4000 50  0001 C CNN
+F 2 "SN74LS161AD:SOIC127P600X175-16N" H 3750 4000 50  0001 C CNN
 F 3 "http://www.ti.com/lit/gpn/sn74LS161" H 3750 4000 50  0001 C CNN
 	1    3750 4000
@@
 F 0 "U7" H 3750 2831 50  0000 C CNN
 F 1 "74LS161" H 3750 2740 50  0000 C CNN
-F 2 "" H 3750 1850 50  0001 C CNN
+F 2 "SN74LS161AD:SOIC127P600X175-16N" H 3750 1850 50  0001 C CNN
 F 3 "http://www.ti.com/lit/gpn/sn74LS161" H 3750 1850 50  0001 C CNN
 	1    3750 1850
@@
 F 0 "U9" H 5300 2831 50  0000 C CNN
 F 1 "74LS161" H 5300 2740 50  0000 C CNN
-F 2 "" H 5300 1850 50  0001 C CNN
+F 2 "SN74LS161AD:SOIC127P600X175-16N" H 5300 1850 50  0001 C CNN
 F 3 "http://www.ti.com/lit/gpn/sn74LS161" H 5300 1850 50  0001 C CNN
 	1    5300 1850
@@
 F 0 "U5" H 2250 2831 50  0000 C CNN
 F 1 "74LS161" H 2250 2740 50  0000 C CNN
-F 2 "" H 2250 1850 50  0001 C CNN
+F 2 "SN74LS161AD:SOIC127P600X175-16N" H 2250 1850 50  0001 C CNN
 F 3 "http://www.ti.com/lit/gpn/sn74LS161" H 2250 1850 50  0001 C CNN
 	1    2250 1850
@@
 F 0 "U10" H 5300 4981 50  0000 C CNN
 F 1 "74LS161" H 5300 4890 50  0000 C CNN
-F 2 "" H 5300 4000 50  0001 C CNN
+F 2 "SN74LS161AD:SOIC127P600X175-16N" H 5300 4000 50  0001 C CNN
 F 3 "http://www.ti.com/lit/gpn/sn74LS161" H 5300 4000 50  0001 C CNN
 	1    5300 4000
@@
 F 0 "U6" H 2250 4981 50  0000 C CNN
 F 1 "74LS161" H 2250 4890 50  0000 C CNN
-F 2 "" H 2250 4000 50  0001 C CNN
+F 2 "SN74LS161AD:SOIC127P600X175-16N" H 2250 4000 50  0001 C CNN
 F 3 "http://www.ti.com/lit/gpn/sn74LS161" H 2250 4000 50  0001 C CNN
 	1    2250 4000

Commit message: added routes
Parts:
- U10, U5, U6, U7, U8, U9: footprint SN74LS161AD:SOIC127P600X175-16N -> Package_DIP:DIP-16_W7.62mm
Changed lines of the file:
@@
 F 0 "U8" H 3750 4981 50  0000 C CNN
 F 1 "74LS161" H 3750 4890 50  0000 C CNN
-F 2 "SN74LS161AD:SOIC127P600X175-16N" H 3750 4000 50  0001 C CNN
+F 2 "Package_DIP:DIP-16_W7.62mm" H 3750 4000 50  0001 C CNN
 F 3 "http://www.ti.com/lit/gpn/sn74LS161" H 3750 4000 50  0001 C CNN
 	1    3750 4000
@@
 F 0 "U7" H 3750 2831 50  0000 C CNN
 F 1 "74LS161" H 3750 2740 50  0000 C CNN
-F 2 "SN74LS161AD:SOIC127P600X175-16N" H 3750 1850 50  0001 C CNN
+F 2 "Package_DIP:DIP-16_W7.62mm" H 3750 1850 50  0001 C CNN
 F 3 "http://www.ti.com/lit/gpn/sn74LS161" H 3750 1850 50  0001 C CNN
 	1    3750 1850
@@
 F 0 "U9" H 5300 2831 50  0000 C CNN
 F 1 "74LS161" H 5300 2740 50  0000 C CNN
-F 2 "SN74LS161AD:SOIC127P600X175-16N" H 5300 1850 50  0001 C CNN
+F 2 "Package_DIP:DIP-16_W7.62mm" H 5300 1850 50  0001 C CNN
 F 3 "http://www.ti.com/lit/gpn/sn74LS161" H 5300 1850 50  0001 C CNN
 	1    5300 1850
@@
 F 0 "U5" H 2250 2831 50  0000 C CNN
 F 1 "74LS161" H 2250 2740 50  0000 C CNN
-F 2 "SN74LS161AD:SOIC127P600X175-16N" H 2250 1850 50  0001 C CNN
+F 2 "Package_DIP:DIP-16_W7.62mm" H 2250 1850 50  0001 C CNN
 F 3 "http://www.ti.com/lit/gpn/sn74LS161" H 2250 1850 50  0001 C CNN
 	1    2250 1850
@@
 F 0 "U10" H 5300 4981 50  0000 C CNN
 F 1 "74LS161" H 5300 4890 50  0000 C CNN
-F 2 "SN74LS161AD:SOIC127P600X175-16N" H 5300 4000 50  0001 C CNN
+F 2 "Package_DIP:DIP-16_W7.62mm" H 5300 4000 50  0001 C CNN
 F 3 "http://www.ti.com/lit/gpn/sn74LS161" H 5300 4000 50  0001 C CNN
 	1    5300 4000
@@
 F 0 "U6" H 2250 4981 50  0000 C CNN
 F 1 "74LS161" H 2250 4890 50  0000 C CNN
-F 2 "SN74LS161AD:SOIC127P600X175-16N" H 2250 4000 50  0001 C CNN
+F 2 "Package_DIP:DIP-16_W7.62mm" H 2250 4000 50  0001 C CNN
 F 3 "http://www.ti.com/lit/gpn/sn74LS161" H 2250 4000 50  0001 C CNN
 	1    2250 4000
