File: vga_controller/vga_controller/pixel_memory.sch (KiCad schematic (older format))
At the start: 9 parts, among them J1 DB15_Female_HighDensity, U11 CAT28C513-D, U12 7400

Commit message: added routes
Parts:
- J1: footprint (none) -> Connector_Dsub:DSUB-15_Female_Horizontal_P2.77x2.54mm_EdgePinOffset9.40mm
- U12: footprint CD4011BE:DIP254P762X508-14 -> Package_DIP:DIP-14_W7.62mm
Changed lines of the file:
@@
 F 0 "J1" H 10350 3217 50  0000 C CNN
 F 1 "DB15_Female_HighDensity" H 10350 3126 50  0000 C CNN
-F 2 "" H 9400 2750 50  0001 C CNN
+F 2 "Connector_Dsub:DSUB-15_Female_Horizontal_P2.77x2.54mm_EdgePinOffset9.40mm" H 9400 2750 50  0001 C CNN
 F 3 " ~" H 9400 2750 50  0001 C CNN
 	1    10350 2350
@@
 F 0 "U12" H 3750 2433 50  0000 C CNN
 F 1 "7400" H 3750 2750 50  0000 C CNN
-F 2 "CD4011BE:DIP254P762X508-14" H 3750 2750 50  0001 C CNN
+F 2 "Package_DIP:DIP-14_W7.62mm" H 3750 2750 50  0001 C CNN
 F 3 "http://www.ti.com/lit/gpn/sn7400" H 3750 2750 50  0001 C CNN
 	1    3750 2750
